Commit message: feat: update navigation sources and README for bngu_2027
Publish only src/ and the root README.md from the current workspace. Includes real and simulation navigation, GICP localization, PGO loop closure, patrol client UI, and real-robot remote-controlled mapping. Preserve actual dependency sources without nested Git metadata or generated build artifacts.

File: src/rm_bnrobot_sim/urdf/bngu_sentinel/base.urdf.xacro (robot description, xacro)
@@ -2,15 +2,9 @@
 <robot xmlns:xacro="http://www.ros.org/wiki/xacro">
     <xacro:include filename="$(find rm_bnrobot_sim)/urdf/bngu_sentinel/common_inertia.xacro" />
-    <!-- 关键修改：参数从 length radius → length width height（长、宽、高独立可控） -->
+    <!-- base_link 直接以地面为 z=0，与实机 TF 定义一致。 -->
     <xacro:macro name="base_xacro" params="length width height">
-        <link name="base_footprint" />
-        <joint name="base_joint" type="fixed">
-            <parent link="base_footprint" />
-            <child link="base_link" />
-            <origin xyz="0.0 0.0 ${height/2.0+0.055-0.008}" rpy="0 0 0" />
-        </joint>
         <link name="base_link">
             <visual>
-                <origin xyz="0 0 0.0" rpy="0 0 0" />
+                <origin xyz="0 0 ${height/2.0+0.055}" rpy="0 0 0" />
                 <geometry>
                     <box size="${length} ${width} ${height}" /> <!-- 长×宽×高 -->
@@ -22,5 +16,5 @@
             <!-- 碰撞：与视觉尺寸一致 -->
             <collision>
-                <origin xyz="0 0 0.0" rpy="0 0 0" />
+                <origin xyz="0 0 ${height/2.0+0.055}" rpy="0 0 0" />
                 <geometry>
                     <box size="${length} ${width} ${height}" />
@@ -30,5 +24,11 @@
                 </material>
             </collision>
-            <xacro:box_inertia m="1.0" w="${length}" h="${width}" d="${height}"/>
+            <inertial>
+                <origin xyz="0 0 ${height/2.0+0.055}" rpy="0 0 0" />
+                <mass value="1.0" />
+                <inertia ixx="${(1.0/12.0) * (width*width + height*height)}" ixy="0.0" ixz="0.0"
+                         iyy="${(1.0/12.0) * (length*length + height*height)}" iyz="0.0"
+                         izz="${(1.0/12.0) * (length*length + width*width)}" />
+            </inertial>
         </link>
     </xacro:macro>

File: src/rm_bnrobot_sim/urdf/bngu_sentinel/bnbot.urdf.xacro (robot description, xacro)
@@ -1,4 +1,5 @@
 <?xml version="1.0"?>
 <robot xmlns:xacro="http://www.ros.org/wiki/xacro" name="bngu_sentinel">
+    <xacro:arg name="cmd_vel_topic" default="cmd_vel" />
     <xacro:include filename="$(find rm_bnrobot_sim)/urdf/bngu_sentinel/base.urdf.xacro" />
     <!-- 传感器组件 -->
@@ -13,15 +14,22 @@
     <xacro:base_xacro length="0.633" width="0.526" height="0.21" />
     <!-- 传感器 -->
-    <xacro:laser_xacro xyz="0 0 0.105" />
-    <!-- 1. Mid360: 相对于base_link的位姿 (extrinsic_T + extrinsic_R) -->
-    <xacro:mid360 name="mid360_laser" topic="/mid360/pointcloud">
-        <origin xyz="0 0 0.6" rpy="${M_PI} 0 ${M_PI/2}" />
+    <xacro:laser_xacro xyz="0 0 0.257" />
+    <!-- Mid-360 FOV 原点：base_link 以地面为 z=0，云台在 URDF 中简化为 base_link。 -->
+    <xacro:mid360 name="mid360" topic="/livox/lidar">
+        <origin xyz="0.22157 0 0.33018" rpy="0 0.7854 0" />
     </xacro:mid360>
-    <!-- 2. IMU: 挂载到mid360_laser_link (而非base_link)，使用相对位姿 -->
-    <joint name="imu_to_mid360_joint" type="fixed">
-        <parent link="mid360_laser_link" />  <!-- Mid360的link名称，需和mid360.urdf.xacro一致 -->
-        <child link="imu_link" />             <!-- IMU的link名称，需和imu.urdf.xacro一致 -->
-        <origin xyz="-0.011 -0.02329 0.04412" rpy="0 0 0" />  <!-- IMU相对于Mid360的位姿 -->
-        <axis xyz="0 0 0" />
+    <!-- 兼容 Livox 驱动的点云 frame id。 -->
+    <link name="livox_frame" />
+    <joint name="mid360_to_livox_frame" type="fixed">
+        <parent link="mid360" />
+        <child link="livox_frame" />
+        <origin xyz="0 0 0" rpy="0 0 0" />
+    </joint>
+    <!-- Mid-360 内置 IMU；与实机 T_base_imu 及 FAST-LIO 配置一致。 -->
+    <link name="livox_imu" />
+    <joint name="base_to_livox_imu" type="fixed">
+        <parent link="base_link" />
+        <child link="livox_imu" />
+        <origin xyz="0.198150552 0.02329 0.291204317" rpy="0 0.7854 0" />
     </joint>
     <!-- <xacro:imu_xacro xyz="0 0 0.02" /> -->
@@ -29,10 +37,10 @@
     <!-- <xacro:imu_xacro xyz="0 0 0.02" /> -->
     <!-- <xacro:camera_xacro xyz="0.10 0 0.45" /> -->
-    <!-- <xacro:mid360 name="mid360_laser" topic="/mid360/pointcloud"> <origin xyz="0.2665 0.0 0.145" rpy="0 0 0" /></xacro:mid360> -->
     <!-- 麦克纳姆轮配置，保持原有轮距参数 -->
-    <xacro:wheel_xacro wheel_name="front_left" xyz="0.235 -0.235 -0.105" yaw="0.7854" axis="-1 1 0" />
-    <xacro:wheel_xacro wheel_name="front_right" xyz="0.235 0.235 -0.105" yaw="2.3562" axis="1 1 0" />
-    <xacro:wheel_xacro wheel_name="rear_left" xyz="-0.235 -0.235 -0.105" yaw="-0.7854" axis="-1 -1 0" />
-    <xacro:wheel_xacro wheel_name="rear_right" xyz="-0.235 0.235 -0.105" yaw="-2.3562" axis="1 -1 0" />
+    <!-- 轮心高度等于轮子半径，避免出生时插入地面造成 IMU 长时间振荡。 -->
+    <xacro:wheel_xacro wheel_name="front_left" xyz="0.235 -0.235 0.055" yaw="0.7854" axis="-1 1 0" />
+    <xacro:wheel_xacro wheel_name="front_right" xyz="0.235 0.235 0.055" yaw="2.3562" axis="1 1 0" />
+    <xacro:wheel_xacro wheel_name="rear_left" xyz="-0.235 -0.235 0.055" yaw="-0.7854" axis="-1 -1 0" />
+    <xacro:wheel_xacro wheel_name="rear_right" xyz="-0.235 0.235 0.055" yaw="-2.3562" axis="1 -1 0" />
     <!-- Gazebo 插件 -->
     <xacro:include filename="$(find rm_bnrobot_sim)/urdf/bngu_sentinel/plugins/gazebo_control_plugin.xacro" />

File: src/rm_bnrobot_sim/urdf/bngu_sentinel/bnbot_real.xacro (robot description, xacro)
@@ -9,9 +9,16 @@
   <xacro:property name="base_mass" value="5.0" />      <!-- 质量(kg) -->
   <xacro:property name="base_center_z" value="${base_height/2}" />  <!-- 底座中心z坐标（自动计算，避免硬编码） -->
-  <!-- 雷达安装参数 -->
-  <xacro:property name="lidar_install_z" value="${base_height}" />  <!-- 雷达安装在底座上表面（z=底座总高度） -->
-  <xacro:property name="lidar_topic" value="mid360" />  <!-- 雷达发布话题（与之前配置一致） -->
-  <!-- 2. 地面参考帧（不变） -->
-  <link name="base_footprint" />
+  <!--
+    实机雷达安装参数。base_link 位于地面零点，并遵循 ROS 的 x 向前、
+    y 向左、z 向上。SolidWorks 导出的 -Z 前向、+Y 向上已转换到 ROS：
+    雷达 FOV 原点向前 221.57 mm、离地 330.18 mm，并向前下方俯 45 度。
+  -->
+  <xacro:property name="lidar_install_x" value="0.22157" />
+  <xacro:property name="lidar_install_y" value="0.0" />
+  <xacro:property name="lidar_install_z" value="0.33018" />
+  <xacro:property name="lidar_install_roll" value="0.0" />
+  <xacro:property name="lidar_install_pitch" value="0.7854" />
+  <xacro:property name="lidar_install_yaw" value="0.0" />
+  <xacro:property name="lidar_topic" value="/livox/lidar" />  <!-- 雷达发布话题（与之前配置一致） -->
   <!-- 3. 核心底座（使用参数化配置） -->
   <link name="base_link">
@@ -40,16 +47,30 @@
     </inertial>
   </link>
-  <!-- 4. base_footprint到base_link的固定关节（参数化z轴高度） -->
-  <joint name="base_joint" type="fixed">
-    <parent link="base_footprint" />
-    <child link="base_link" />
-    <origin xyz="0.0 0.0 ${base_center_z}" rpy="0 0 0" />  <!-- z=底座中心高度（下表面贴地） -->
-  </joint>
-  <!-- 5. 集成Livox Mid360激光雷达（保持原有宏调用，参数化配置） -->
+  <!-- 4. 集成 Livox Mid-360；实机 TF 根节点直接使用 base_link。 -->
   <!-- 包含Mid360的xacro文件（确保ros2_livox_simulation功能包已编译安装） -->
   <xacro:include filename="$(find ros2_livox_simulation)/urdf/mid360.xacro" />
   <!-- 调用Mid360宏：使用参数化安装位置和话题 -->
   <xacro:mid360 name="mid360" parent="base_link" topic="${lidar_topic}" >
-    <origin xyz="0 0 ${lidar_install_z}" rpy="0 0 0"/>
+    <origin xyz="${lidar_install_x} ${lidar_install_y} ${lidar_install_z}"
+            rpy="${lidar_install_roll} ${lidar_install_pitch} ${lidar_install_yaw}"/>
   </xacro:mid360>
+  <!-- livox_ros_driver2 的原始点云和 IMU 消息使用该兼容 frame id。 -->
+  <link name="livox_frame" />
+  <joint name="mid360_to_livox_frame" type="fixed">
+    <parent link="mid360" />
+    <child link="livox_frame" />
+    <origin xyz="0 0 0" rpy="0 0 0" />
+  </joint>
+  <!--
+    Mid-360 内置 IMU 原点。这里由 T_base_lidar 和 FAST-LIO 官方
+    T_imu_lidar (R=I, t=[-0.011,-0.02329,0.04412]) 组合得到。
+    p_base = R_base_imu * p_imu + t_base_imu。
+  -->
+  <link name="livox_imu" />
+  <joint name="base_to_livox_imu" type="fixed">
+    <parent link="base_link" />
+    <child link="livox_imu" />
+    <origin xyz="0.198150552 0.02329 0.291204317"
+            rpy="${lidar_install_roll} ${lidar_install_pitch} ${lidar_install_yaw}" />
+  </joint>
 </robot>

File: src/rm_bnrobot_sim/urdf/bngu_sentinel/plugins/gazebo_control_plugin.xacro (robot description, xacro)
@@ -6,5 +6,5 @@
                 <ros>
                     <namespace>/</namespace>
-                    <remapping>cmd_vel:=cmd_vel</remapping>
+                    <remapping>cmd_vel:=$(arg cmd_vel_topic)</remapping>
                     <remapping>odom:=odom</remapping>
                 </ros>
@@ -27,5 +27,6 @@
                 <publish_odom_tf>false</publish_odom_tf>
                 <odometry_frame>odom</odometry_frame>
-                <robot_base_frame>base_footprint</robot_base_frame>
+                <!-- odom -> base_link 由 FAST-LIO 发布，Gazebo 只发布里程计消息。 -->
+                <robot_base_frame>base_link</robot_base_frame>
             </plugin>
         </gazebo>

File: src/rm_bnrobot_sim/urdf/bngu_sentinel/plugins/gazebo_sensor_plugin.xacro (robot description, xacro)
@@ -7,5 +7,6 @@
                     <ros>
                         <namespace>/</namespace>
-                        <remapping>~/out:=scan</remapping>
+                        <!-- 保留调试用 2D 雷达，避免与 Mid-360 切片的 /scan 冲突。 -->
+                        <remapping>~/out:=scan_2d_raw</remapping>
                     </ros>
                     <output_type>sensor_msgs/LaserScan</output_type>
@@ -43,10 +44,10 @@
             </sensor>
         </gazebo>
-<gazebo reference="imu_link">
+<gazebo reference="livox_imu">
     <sensor name="imu_sensor" type="imu">
         <plugin name="imu_plugin" filename="libgazebo_ros_imu_sensor.so">
             <ros>
                 <namespace>/</namespace>
-                <remapping>~/out:=imu</remapping>
+                <remapping>~/out:=livox/imu</remapping>
             </ros>
             <initial_orientation_as_reference>false</initial_orientation_as_reference>

File: src/rm_bnrobot_sim/urdf/bngu_sentinel/sensor/mid360.urdf.xacro (robot description, xacro)
@@ -10,7 +10,9 @@
   <xacro:property name="laser_min_range" value="0.1" /> <!-- 最小探测距离（m） -->
   <xacro:property name="laser_max_range" value="200.0" /> <!-- 最大探测距离（m） -->
-  <xacro:property name="laser_update_rate" value="20" /> <!-- 刷新频率（Hz），Mid360最大支持20Hz -->
-  <xacro:property name="horizontal_samples" value="300" /> <!-- 水平采样数（越多数据越密） -->
-  <xacro:property name="vertical_samples" value="64" /> <!-- 垂直采样数（Mid360实际为64线） -->
+  <xacro:property name="laser_update_rate" value="10" /> <!-- 与实机驱动默认 publish_freq=10 Hz 一致。 -->
+  <!-- Gazebo ray casting is much heavier than the real sensor. This density
+       preserves the Mid-360 scan pattern while keeping the GUI responsive. -->
+  <xacro:property name="horizontal_samples" value="150" />
+  <xacro:property name="vertical_samples" value="32" />
   <xacro:property name="horizontal_min_angle" value="0" /> <!-- 水平最小角度（弧度） -->
   <xacro:property name="horizontal_max_angle" value="${2*M_PI}" /> <!-- 水平最大角度（360°） -->
@@ -20,7 +22,7 @@
   <xacro:property name="noise_mean" value="0.0" /> <!-- 噪声均值 -->
   <xacro:property name="noise_stddev" value="0.002" /> <!-- 噪声标准差 -->
-  <xacro:property name="downsample_rate" value="2" /> <!-- 降采样系数（2=每2个点保留1个） -->
+  <xacro:property name="downsample_rate" value="8" /> <!-- 每 20000 个扫描位置保留 2500 条射线，避免只截取短段垂直扫描。 -->
   <!-- 2. 雷达模型-->
-  <xacro:macro name="mid360" params=" name:='mid360_laser' parent:='base_link' topic:='/mid360/pointcloud' *origin">
+  <xacro:macro name="mid360" params="name:='mid360' parent:='base_link' topic:='/livox/lidar' *origin">
     <link name="${name}">
       <visual>
@@ -28,5 +30,5 @@
         <origin xyz="0.025 -0.0265 -0.025" rpy="${M_PI/2} 0 ${M_PI}"/>
         <geometry>
-          <mesh filename="file:///home/mage/navigation/nav_RM_4/src/rm_bnrobot_sim/meshes/mid360.stl" scale="0.0008 0.0008 0.0008"/>
+          <mesh filename="file://$(find rm_bnrobot_sim)/meshes/mid360.stl" scale="0.0008 0.0008 0.0008"/>
         </geometry>
         <material name="black">
@@ -57,9 +59,12 @@
         <!-- <pose>0 0 0 0 0 0</pose>  -->
         <pose>0.0 0.0 0.0 0 0</pose><!-- 传感器自身在link中的姿态（无偏移） -->
-        <visualize>true</visualize> <!-- 在Gazebo中显示扫描线（调试用） -->
+        <always_on>true</always_on>
+        <!-- Thousands of rendered rays can make gzclient consume several GB. -->
+        <visualize>false</visualize>
         <update_rate>${laser_update_rate}</update_rate> <!-- 刷新频率 -->
         <!-- 6. Livox雷达插件（发布点云数据） -->
         <plugin name="${name}_plugin" filename="libros2_livox.so">
           <simulate>true</simulate>
+          <frame_name>livox_frame</frame_name>
           <ray>
             <scan>
@@ -93,7 +98,9 @@
           </ray>
           <visualize>false</visualize> <!-- 点云可视化由RViz负责，Gazebo中关闭 -->
-          <samples>${horizontal_samples * vertical_samples}</samples> <!-- 总采样数 -->
+          <!-- Advance a complete 0.1 s pattern interval, retaining about the same
+               ray count as before (2500 instead of 2400). -->
+          <samples>20000</samples>
           <downsample>${downsample_rate}</downsample> <!-- 降采样 -->
-          <csv_file_name>$(find rm_bnrobot_sim)/scan_mode/mid360.csv</csv_file_name> 扫描模式配置文件
+          <csv_file_name>$(find rm_bnrobot_sim)/scan_mode/mid360.csv</csv_file_name>
           <topic>${topic}</topic> <!-- 点云发布话题 -->
         </plugin>
