Commit message: 除下发外完整导航链路（实机通过）

File: src/rm_bnrobot_sim/urdf/bngu_sentinel/bnbot.urdf.xacro (robot description, xacro)
@@ -15,7 +15,8 @@
     <!-- 传感器 -->
     <xacro:laser_xacro xyz="0 0 0.257" />
-    <!-- Mid-360 FOV 原点：base_link 以地面为 z=0，云台在 URDF 中简化为 base_link。 -->
+    <!-- Mid-360 FOV 原点：车体左侧 0.22157 m，无前向偏移；base_link 以地面为 z=0。
+         雷达 x 轴向前，z 轴向左上方，沿用约 45 度倾角（roll=-0.7854）。 -->
     <xacro:mid360 name="mid360" topic="/livox/lidar">
-        <origin xyz="0.22157 0 0.33018" rpy="0 0.7854 0" />
+        <origin xyz="0 0.22157 0.33018" rpy="-0.7854 0 0" />
     </xacro:mid360>
     <!-- 兼容 Livox 驱动的点云 frame id。 -->
@@ -31,5 +32,5 @@
         <parent link="base_link" />
         <child link="livox_imu" />
-        <origin xyz="0.198150552 0.02329 0.291204317" rpy="0 0.7854 0" />
+        <origin xyz="0.011000000 0.206840878 0.282513959" rpy="-0.7854 0 0" />
     </joint>
     <!-- <xacro:imu_xacro xyz="0 0 0.02" /> -->

File: src/rm_bnrobot_sim/urdf/bngu_sentinel/bnbot_real.xacro (robot description, xacro)
@@ -12,11 +12,12 @@
     实机雷达安装参数。base_link 位于地面零点，并遵循 ROS 的 x 向前、
     y 向左、z 向上。SolidWorks 导出的 -Z 前向、+Y 向上已转换到 ROS：
-    雷达 FOV 原点向前 221.57 mm、离地 330.18 mm，并向前下方俯 45 度。
+    雷达 FOV 原点位于车体左侧 221.57 mm，无前向偏移，离地 330.18 mm，
+    雷达 x 轴向前，z 轴向左上方（沿用约 45 度倾角，roll=-0.7854）。
   -->
-  <xacro:property name="lidar_install_x" value="0.22157" />
-  <xacro:property name="lidar_install_y" value="0.0" />
+  <xacro:property name="lidar_install_x" value="0.0" />
+  <xacro:property name="lidar_install_y" value="0.22157" />
   <xacro:property name="lidar_install_z" value="0.33018" />
-  <xacro:property name="lidar_install_roll" value="0.0" />
-  <xacro:property name="lidar_install_pitch" value="0.7854" />
+  <xacro:property name="lidar_install_roll" value="-0.7854" />
+  <xacro:property name="lidar_install_pitch" value="0.0" />
   <xacro:property name="lidar_install_yaw" value="0.0" />
   <xacro:property name="lidar_topic" value="/livox/lidar" />  <!-- 雷达发布话题（与之前配置一致） -->
@@ -71,5 +72,5 @@
     <parent link="base_link" />
     <child link="livox_imu" />
-    <origin xyz="0.198150552 0.02329 0.291204317"
+    <origin xyz="0.011000000 0.206840878 0.282513959"
             rpy="${lidar_install_roll} ${lidar_install_pitch} ${lidar_install_yaw}" />
   </joint>
